Commit message: Change pitch_joint type to continuous

File: urdf/rm_gimbal.urdf.xacro (robot description, xacro)
@@ -13,5 +13,5 @@
   </joint>
   <link name="pitch_link" />
-  <joint name="pitch_joint" type="revolute">
+  <joint name="pitch_joint" type="continuous">
     <parent link="yaw_link" />
     <child link="pitch_link" />

Commit message: Change xyz & rpy to args

File: urdf/rm_gimbal.urdf.xacro (robot description, xacro)
@@ -2,7 +2,6 @@
 <robot name="rm_gimbal"
   xmlns:xacro="http://ros.org/wiki/xacro">
-  <xacro:property name="gimbal_camera_transfrom">
-    <origin xyz="0.10 0 0.05" rpy="0 0 0" />
-  </xacro:property>
+  <xacro:arg name="xyz" default="0.10 0 0.05" />
+  <xacro:arg name="rpy" default="0 0 0" />
   <link name="odom" />
   <link name="yaw_link" />
@@ -20,5 +19,5 @@
   <link name="camera_link" />
   <joint name="camera_joint" type="fixed">
-    <xacro:insert_block name="gimbal_camera_transfrom" />
+    <origin xyz="$(arg xyz)" rpy="$(arg rpy)" />
     <parent link="pitch_link" />
     <child link="camera_link" />

Commit message: Using floating joint

File: urdf/rm_gimbal.urdf.xacro (robot description, xacro)
@@ -5,20 +5,13 @@
   <xacro:arg name="rpy" default="0 0 0" />
   <link name="odom" />
-  <link name="yaw_link" />
-  <joint name="yaw_joint" type="continuous">
+  <link name="gimbal_link" />
+  <joint name="gimbal_joint" type="floating">
     <parent link="odom" />
-    <child link="yaw_link" />
-    <axis xyz="0 0 1" />
-  </joint>
-  <link name="pitch_link" />
-  <joint name="pitch_joint" type="continuous">
-    <parent link="yaw_link" />
-    <child link="pitch_link" />
-    <axis xyz="0 1 0" />
+    <child link="gimbal_link" />
   </joint>
   <link name="camera_link" />
   <joint name="camera_joint" type="fixed">
     <origin xyz="$(arg xyz)" rpy="$(arg rpy)" />
-    <parent link="pitch_link" />
+    <parent link="gimbal_link" />
     <child link="camera_link" />
     <axis xyz="0 0 0" />
